Commit message: V1.1,added Gazebo launch file and xacro description

File: crp09/urdf/my_crp09.urdf (robot description, URDF)
Before this commit: robot my_crp09, 2 links, 1 joints
Links:
- removed link pan_link
- added link bottom_link; collision box size=1 1 0.02; visual box size=1 1 0.02
- added link gripper_finger1, mass 1; collision box size=0.01 0.01 0.04; visual box size=0.01 0.01 0.04
- added link gripper_finger2, mass 1; collision box size=0.01 0.01 0.04; visual box size=0.01 0.01 0.04
- added link link1, mass 1; collision cylinder length=0.171 radius=0.1125; visual cylinder length=0.171 radius=0.1125
- added link link2, mass 1; collision cylinder length=0.455 radius=0.1; visual cylinder length=0.455 radius=0.1
- added link link3, mass 1; collision cylinder length=0.15 radius=0.04; visual cylinder length=0.15 radius=0.04
- added link link4, mass 1; collision cylinder length=0.29 radius=0.04; visual cylinder length=0.29 radius=0.04
- added link link5, mass 1; collision cylinder length=0.105 radius=0.04; visual cylinder length=0.105 radius=0.04
- added link link_tool, mass 1; collision cylinder length=0.02 radius=0.035; visual cylinder length=0.02 radius=0.035
Joints:
- removed joint pan_joint
- added joint bottom_joint: type fixed, parent base_link, child bottom_link, origin xyz=0 0 0 rpy=0 0 0
- added joint finger_joint1: type prismatic, parent link_tool, child gripper_finger1, origin xyz=0 0.02 0.035, axis 0 0 1, limit lower=-0.03 upper=0 effort=300 velocity=0.1
- added joint finger_joint2: type prismatic, parent link_tool, child gripper_finger2, origin xyz=0 0.02 -0.035, axis 0 0 1, limit lower=0 upper=0.03 effort=300 velocity=0.1
- added joint joint1: type revolute, parent base_link, child link1, origin xyz=0 0 0.25, axis 0 0 1, limit lower=-2.96 upper=2.96 effort=300 velocity=0.1
- added joint joint2: type revolute, parent link1, child link2, origin xyz=0 0 0.171, axis 1 0 0, limit lower=-2.355 upper=1.74 effort=300 velocity=0.1
- added joint joint3: type revolute, parent link2, child link3, origin xyz=0 0 0.455, axis 1 0 0, limit lower=-1.13 upper=3.05 effort=300 velocity=0.1
- added joint joint4: type revolute, parent link3, child link4, origin xyz=0 0.15 0, axis 0 1 0, limit lower=-2.96 upper=2.96 effort=300 velocity=0.1
- added joint joint5: type revolute, parent link4, child link5, origin xyz=0 0.29 0, axis 1 0 0, limit lower=-2.093 upper=2.093 effort=300 velocity=0.1
- added joint joint6: type revolute, parent link5, child link_tool, origin xyz=0 0.105 0, axis 0 1 0, limit lower=-3.14 upper=3.14 effort=300 velocity=0.1

File: crp09/urdf/my_crp09.xacro (robot description, xacro)
@@ -1,4 +1,63 @@
 <?xml version="1.0"?>
-<robot name="crp09">
+<robot name="my_crp09" xmlns:xacro="http://ros.org/wiki/xacro">
+  <!-- Include materials -->
+    <material name="Black">
+        <color rgba="0.0 0.0 0.0 1.0"/>
+    </material>
+    <material name="Red">
+        <color rgba="0.8 0.0 0.0 1.0"/>
+    </material>
+    <material name="White">
+        <color rgba="1.0 1.0 1.0 1.0"/>
+    </material>
+  <xacro:property name="deg_to_rad" value="0.01745329251994329577"/>
+  <!-- Constants -->
+  <xacro:property name="M_SCALE" value="0.001 0.001 0.001"/>
+  <xacro:property name="M_PI" value="3.14159"/>
+   <xacro:macro name="inertial_matrix" params="mass">
+      <inertial>
+      	<mass value="${mass}" />
+        <inertia ixx="1.0" ixy="0.0" ixz="0.0" iyy="0.5" iyz="0.0" izz="1.0" />
+      </inertial>
+   </xacro:macro>
+   <xacro:macro name="transmission_block" params="joint_name">
+	  <transmission name="tran1">
+	    <type>transmission_interface/SimpleTransmission</type>
+	    <joint name="${joint_name}">
+	      <hardwareInterface>hardware_interface/PositionJointInterface</hardwareInterface>
+	    </joint>
+	    <actuator name="motor1">
+	      <hardwareInterface>hardware_interface/PositionJointInterface</hardwareInterface>
+	      <mechanicalReduction>1</mechanicalReduction>
+	    </actuator>
+	  </transmission>
+   </xacro:macro>
+<!-- BOTTOM FIXED LINK
+This link is the base of the arm in which arm is placed
+-->
+<!-- ///////////////////////////////////////////////////////////////////////////////////////////////////////////////////// -->
+  <joint name="bottom_joint" type="fixed">
+    <origin xyz="0 0 0" rpy="0 0 0" />
+    <parent link="base_link"/>
+    <child link="bottom_link"/>
+  </joint>
+  <link name="bottom_link">
+    <visual>
+      <origin xyz=" 0 0 -0.01"  rpy="0 0 0"/>
+      <geometry>
+	       <box size="1 1 0.02" />
+      </geometry>
+      <material name="Brown" />
+    </visual>
+    <collision>
+      <origin xyz=" 0 0 -0.01"  rpy="0 0 0"/>
+      <geometry>
+	       <box size="1 1 0.02" />
+      </geometry>
+      </collision>>
+  </link>
+  <gazebo reference="bottom_link">
+    <material>Gazebo/Red</material>
+  </gazebo>
   <link name="base_link">
     <visual>
@@ -22,5 +81,5 @@
     </inertial>
   <gazebo reference="base_link">
-    <material>Gazebo/Blue</material>
+    <material>Gazebo/White</material>
   </gazebo>
   </link>
@@ -54,5 +113,5 @@
     </inertial>
   <gazebo reference="link1">
-    <material>Gazebo/Blue</material>
+    <material>Gazebo/Red</material>
   </gazebo>
   </link>
@@ -86,5 +145,5 @@
     </inertial>
   <gazebo reference="link2">
-    <material>Gazebo/Blue</material>
+    <material>Gazebo/White</material>
   </gazebo>
   </link>
@@ -118,5 +177,5 @@
     </inertial>
   <gazebo reference="link3">
-    <material>Gazebo/Blue</material>
+    <material>Gazebo/Red</material>
   </gazebo>
   </link>
@@ -150,5 +209,5 @@
     </inertial>
   <gazebo reference="link4">
-    <material>Gazebo/Blue</material>
+    <material>Gazebo/White</material>
   </gazebo>
   </link>
@@ -182,5 +241,5 @@
     </inertial>
   <gazebo reference="link5">
-    <material>Gazebo/Blue</material>
+    <material>Gazebo/Red</material>
   </gazebo>
   </link>
@@ -215,5 +274,5 @@
     </inertial>
   <gazebo reference="link_tool">
-    <material>Gazebo/Blue</material>
+    <material>Gazebo/White</material>
   </gazebo>
   </link>
@@ -247,5 +306,5 @@
     </inertial>
   <gazebo reference="gripper_finger1">
-    <material>Gazebo/Blue</material>
+    <material>Gazebo/White</material>
   </gazebo>
   </link>
@@ -279,6 +338,22 @@
     </inertial>
   <gazebo reference="gripper_finger2">
-    <material>Gazebo/Blue</material>
-  </gazebo>
-  </link>
+    <material>Gazebo/White</material>
+  </gazebo>
+  </link>
+<!-- ///////////////////////////////////////////////////////////////////////////////////////////////////////////////////// -->
+  <!-- Transmissions for ROS Control -->
+   <xacro:transmission_block joint_name="joint1"/>
+   <xacro:transmission_block joint_name="joint2"/>
+   <xacro:transmission_block joint_name="joint3"/>
+   <xacro:transmission_block joint_name="joint4"/>
+   <xacro:transmission_block joint_name="joint5"/>
+   <xacro:transmission_block joint_name="joint6"/>
+   <xacro:transmission_block joint_name="finger_joint1"/>
+   <xacro:transmission_block joint_name="finger_joint2"/>
+ <!-- ros_control plugin -->
+  <gazebo>
+    <plugin name="gazebo_ros_control" filename="libgazebo_ros_control.so">
+      <robotNamespace>/my_crp09</robotNamespace>
+    </plugin>
+  </gazebo>
 </robot>
