Commit message: 改为差速驱动

File: my_car/urdf/my_car.urdf (robot description, URDF)
Before this commit: robot my_car, 5 links, 4 joints
Links:
- removed link left_front_wheel
- removed link right_front_wheel
- added link caster_wheel, mass 1; collision cylinder length=.02 radius=0.0375; visual cylinder length=.02 radius=0.0375
- added link hokuyo_link; visual box size=0.05 0.05 0.05
- link left_back_wheel: geometry collision cylinder length=.02 radius=0.1; visual cylinder length=.02 radius=0.1
- link right_back_wheel: geometry collision cylinder length=.02 radius=0.1; visual cylinder length=.02 radius=0.1
Joints:
- removed joint left_front_wheel_joint
- removed joint right_front_wheel_joint
- added joint caster_wheel_joint: type fixed, parent base_link, child caster_wheel, origin xyz=0 0.45 0.0375 rpy=0 -1.57075 0
- added joint hokuyo_joint: type fixed, parent base_link, child hokuyo_link, origin xyz=0 0.45 0.125 rpy=0 0 0
- joint left_back_wheel_joint: origin xyz=-0.375 -0.45 0.075 rpy=0 -1.57075 0 -> xyz=-0.375 -0.45 0.1 rpy=0 -1.57075 0
- joint right_back_wheel_joint: origin xyz=0.375 -0.45 0.075 rpy=0 -1.57075 0 -> xyz=0.375 -0.45 0.1 rpy=0 -1.57075 0

Commit message: 四轮差速，待完善

File: my_car/urdf/my_car.urdf (robot description, URDF)
Before this commit: robot my_car, 5 links, 4 joints
Links:
- removed link caster_wheel
- added link left_front_wheel, mass 1; collision cylinder length=.02 radius=0.075; visual cylinder length=.02 radius=0.075
- added link right_front_wheel, mass 1; collision cylinder length=.02 radius=0.075; visual cylinder length=.02 radius=0.075
- link left_back_wheel: geometry collision cylinder length=.02 radius=0.075; visual cylinder length=.02 radius=0.075
- link right_back_wheel: geometry collision cylinder length=.02 radius=0.075; visual cylinder length=.02 radius=0.075
Joints:
- removed joint caster_wheel_joint
- added joint left_front_wheel_joint: type continuous, parent base_link, child left_front_wheel, origin xyz=-0.375 0.45 0.075 rpy=0 -1.57075 0, axis 0 0 1, limit effort=100 velocity=100
- added joint right_front_wheel_joint: type continuous, parent base_link, child right_front_wheel, origin xyz=0.375 0.45 0.075 rpy=0 -1.57075 0, axis 0 0 1, limit effort=100 velocity=100
- joint hokuyo_joint: origin xyz=0 0.45 0.125 rpy=0 0 0 -> xyz=0 0.45 0.1 rpy=0 0 0
- joint left_back_wheel_joint: origin xyz=-0.375 -0.45 0.1 rpy=0 -1.57075 0 -> xyz=-0.375 -0.45 0.075 rpy=0 -1.57075 0
- joint right_back_wheel_joint: origin xyz=0.375 -0.45 0.1 rpy=0 -1.57075 0 -> xyz=0.375 -0.45 0.075 rpy=0 -1.57075 0

Commit message: 小车建模

File: my_car/urdf/my_car.urdf (robot description, URDF)
Before this commit: robot my_car, 5 links, 4 joints
Links:
- removed link caster_wheel
- added link caster_wheel_back, mass 1; collision cylinder length=.02 radius=0.0375; visual cylinder length=.02 radius=0.0375
- added link caster_wheel_front, mass 1; collision cylinder length=.02 radius=0.0375; visual cylinder length=.02 radius=0.0375
Joints:
- removed joint caster_wheel_joint
- added joint caster_wheel_back_joint: type fixed, parent base_link, child caster_wheel_back, origin xyz=0 -0.45 0.0375 rpy=0 -1.57075 0
- added joint caster_wheel_front_joint: type fixed, parent base_link, child caster_wheel_front, origin xyz=0 0.45 0.0375 rpy=0 -1.57075 0

Commit message: 使用PI控制角度

File: my_car/urdf/my_car.urdf (robot description, URDF)
Before this commit: robot my_car, 6 links, 5 joints
Links:
- link base_link: mass 10 -> 50
Joints:
- joint left_back_wheel_joint: origin xyz=-0.25 -0.25 0.075 rpy=0 -1.57075 0 -> xyz=-0.25 0 0.075 rpy=0 -1.57075 0
- joint right_back_wheel_joint: origin xyz=0.25 -0.25 0.075 rpy=0 -1.57075 0 -> xyz=0.25 0 0.075 rpy=0 -1.57075 0
